File: PCB/range_selector.kicad_sch (KiCad schematic)
At the start: 24 parts, among them U201 74HC14, U202 74HC00, U4 74HC193, U5 74HC139, U6 74HC14

Commit message: schematic roughly done
Parts:
- D201, D202, D203, D204: value LED -> LED_R
Other:
- note added: "Counter"
- note added: "Debouncer"
- note added: "Decoder"
- moved on the sheet: C10, C11, C12, C13, C201, C202, D201, R10, R11, R201, R202, R203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

Commit message: footprints
Parts:
- C201: footprint (none) -> Capacitor_SMD:C_0603_1608Metric
- C202: renamed from C12; footprint (none) -> Capacitor_SMD:C_0603_1608Metric
- C203: renamed from C13; footprint (none) -> Capacitor_SMD:C_0603_1608Metric
- C204: renamed from C202; footprint (none) -> Capacitor_SMD:C_0603_1608Metric
- C205: renamed from C10; footprint (none) -> Capacitor_SMD:C_0603_1608Metric
- C206: renamed from C11; footprint (none) -> Capacitor_SMD:C_0603_1608Metric
- D201, D202, D203, D204: footprint (none) -> LED_SMD:LED_0603_1608Metric
- R201: renamed from R8; footprint (none) -> Resistor_SMD:R_0603_1608Metric
- R202: renamed from R10; footprint (none) -> Resistor_SMD:R_0603_1608Metric
- R203: renamed from R9; footprint (none) -> Resistor_SMD:R_0603_1608Metric
- R204: renamed from R11; footprint (none) -> Resistor_SMD:R_0603_1608Metric
- R205: renamed from R7; footprint (none) -> Resistor_SMD:R_0603_1608Metric
- R206: renamed from R201; footprint (none) -> Resistor_SMD:R_0603_1608Metric
- R207: renamed from R202; footprint (none) -> Resistor_SMD:R_0603_1608Metric
- R208: renamed from R203; footprint (none) -> Resistor_SMD:R_0603_1608Metric
- R209: renamed from R204; footprint (none) -> Resistor_SMD:R_0603_1608Metric
- U201, U202: footprint (none) -> w-ic:SOIC-14 208mil
- U201: renamed from U6; footprint (none) -> w-ic:SOIC-14 208mil
- renumbered U4 to U203, U5 to U204
Other:
- moved on the sheet: D201, D202, D203, D204, R206, R207, R208, R209

Commit message: changes
Parts:
- removed U201: 74HC14, w-ic:SOIC-14 208mil, symbol 74xx:74HC14
- removed U202: 74HC00, w-ic:SOIC-14 208mil, symbol 74xx:74HC00
- added U106: 74HC00, w-ic:SOIC-14 3.9x8.6mm P1.27mm, symbol 74xx:74HC00
- added U203: 74HC14, w-ic:SOIC-14 3.9x8.6mm P1.27mm, symbol 74xx:74HC14
- renumbered U203 to U201, U204 to U202
Connections:
- net +5V: now also U106.14 (VCC), U203.14 (VCC)
- net CT_DOWN: now also U106.6
- net CT_UP: now also U106.3
- net GND: now also U106.7 (GND), U203.7 (GND)
- net R1: now also U106.4, U203.6
- net R2: now also U203.8
- net R3: now also U203.10
- net R4: now also U106.2, U203.12
- net at C202.1, R203.2: now also U203.1
- net at U202.4 (~{1Y0}): now also U203.5
- net at C203.1, R204.2: now also U203.3
- net at U202.7 (~{1Y3}): now also U203.13
- net at U202.6 (~{1Y2}): now also U203.11
- net at U202.5 (~{1Y1}): now also U203.9
- new net: U106.1, U203.2
- new net: U106.5, U203.4

Commit message: start of layout
Parts:
- removed R205: 10k, Resistor_SMD:R_0603_1608Metric, symbol Device:R
- D201, D202, D203, D204: footprint LED_SMD:LED_0603_1608Metric -> LED_THT:LED_D3.0mm
Connections:
- net +5V: now also U201.11 (~{LOAD}), U202.15 (~{E2})
- net GND: no longer U202.15 (~{E2})
- net R1: no longer U106.4
- net R4: no longer U106.2
- net at U202.4 (~{1Y0}), U203.5: now also U106.4
- net at U202.7 (~{1Y3}), U203.13: now also U106.2
Other:
- note added: "0/1"
- note added: "1/0"
- moved on the sheet: C202, C203, D201, D202, D203, D204, R201, R202, R203, R204, R206, R207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
