File: PCB/PCB.kicad_sch (KiCad schematic)
At the start: 31 parts, among them J101 Current_input, J102 Banana conn. red, J103 Banana conn. black, J104 Conn_Coaxial, Q101 BC817, Q102 BC817, Q103 BC817, Q104 BC817, SW101 SW_Push, SW102 SW_Push, U101 TSV782, U102 OJ-SH-105HM, U103 OJ-SH-105HM, U104 OJ-SH-105HM, U105 OJ-SH-105HM

Commit message: rough layout done
Parts:
- J101: footprint TerminalBlock_Phoenix:TerminalBlock_Phoenix_MPT-0,5-2-2.54_1x02_P2.54mm_Horizontal -> w-connector:Terminal Block 2x3,5mm
- SW101, SW102: footprint Connector_PinHeader_2.54mm:PinHeader_1x02_P2.54mm_Vertical -> Button_Switch_THT:SW_Tactile_SPST_Angled_PTS645Vx83-2LFS
Changed lines of the file:
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@@
 			)
 		)
-		(property "Footprint" "Connector_PinHeader_2.54mm:PinHeader_1x02_P2.54mm_Vertical"
+		(property "Footprint" "Button_Switch_THT:SW_Tactile_SPST_Angled_PTS645Vx83-2LFS"
 			(at 71.12 134.62 0)
 			(effects
@@
 			)
 		)
-		(property "Footprint" "Connector_PinHeader_2.54mm:PinHeader_1x02_P2.54mm_Vertical"
+		(property "Footprint" "Button_Switch_THT:SW_Tactile_SPST_Angled_PTS645Vx83-2LFS"
 			(at 71.12 149.86 0)
 			(effects
@@
 			)
 		)
-		(property "Footprint" "TerminalBlock_Phoenix:TerminalBlock_Phoenix_MPT-0,5-2-2.54_1x02_P2.54mm_Horizontal"
+		(property "Footprint" "w-connector:Terminal Block 2x3,5mm"
 			(at 82.55 41.91 0)
 			(effects

Commit message: changed BNC footprint
Parts:
- J104: footprint w-connector:GOLDEN LOCH 900D-6452R2 -> Connector_Coaxial:BNC_Amphenol_B6252HB-NPP3G-50_Horizontal
Changed lines of the file:
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@@
 			)
 		)
-		(property "Footprint" "w-connector:GOLDEN LOCH 900D-6452R2"
+		(property "Footprint" "Connector_Coaxial:BNC_Amphenol_B6252HB-NPP3G-50_Horizontal"
 			(at 346.71 105.41 0)
 			(effects
